File: board/RCMx1_v04/RCMx1 Rev_04.brd (EAGLE design)
At the start: 86.5 x 78.7 mm, 74 parts, among them J1 CON_2X2_0_100, J12 CON2X2, J14 CON2X2, J15 CON2X2, J16 CON1X18, J2 CON_2X2_0_100, J20 CON_3X17_0_100, J3 CON_2X16_0_100, J6 CON_3X17_0_100, J8 M05X2PTH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

Commit message: Rotated board name on top silk layer 180 degrees.
Parts:
- removed U$5: (no value), SparkFun-Aesthetics:OSHW-LOGO-M
- added LOGO3: OSHW-LOGOM, SparkFun-Aesthetics:OSHW-LOGO-M
Other:
- board text added: "E^3 RCMx1 v4"
- board text removed: "RCMx1 v4"
Changed lines of the file:
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@@
 <layer number="20" name="Dimension" color="15" fill="1" visible="yes" active="yes"/>
 <layer number="21" name="tPlace" color="7" fill="1" visible="yes" active="yes"/>
-<layer number="22" name="bPlace" color="7" fill="1" visible="no" active="yes"/>
+<layer number="22" name="bPlace" color="7" fill="1" visible="yes" active="yes"/>
 <layer number="23" name="tOrigins" color="15" fill="1" visible="yes" active="yes"/>
-<layer number="24" name="bOrigins" color="15" fill="1" visible="no" active="yes"/>
+<layer number="24" name="bOrigins" color="15" fill="1" visible="yes" active="yes"/>
 <layer number="25" name="tNames" color="7" fill="1" visible="no" active="yes"/>
 <layer number="26" name="bNames" color="7" fill="1" visible="no" active="yes"/>
@@
 <text x="72.898" y="6.858" size="1.27" layer="21" rot="SR0.6">SCL</text>
 <text x="72.771" y="4.191" size="1.27" layer="21" rot="SR0">GND</text>
-<text x="0.889" y="39.243" size="2.54" layer="21" rot="SR270">RCMx1 v4</text>
+<text x="3.0734" y="17.526" size="2.286" layer="21" rot="SR90">E^3 RCMx1 v4</text>
 <text x="3.81" y="52.324" size="2.54" layer="21" font="vector" ratio="14" rot="R90">-</text>
 <text x="4.2164" y="52.07" size="2.54" layer="21">+</text>
@@
 <wire x1="72.39" y1="11.43" x2="72.39" y2="14.605" width="0.254" layer="21"/>
 <text x="72.136" y="13.716" size="1.6764" layer="21" font="vector" rot="R180">I2C</text>
-<text x="1.524" y="51.3588" size="1.778" layer="21" rot="SR270">PWR IN</text>
+<text x="1.524" y="51.3588" size="1.524" layer="21" rot="SR270">PWR IN</text>
 <text x="78.994" y="47.371" size="1.016" layer="21" font="vector" ratio="12" rot="SR90">UART1</text>
 <text x="81.534" y="40.005" size="1.016" layer="21" font="vector" ratio="12" rot="SR90">FLOW</text>
@@
 <element name="U$2" library="JLY Parts" package="GNDPAD" value="GNDPAD" x="3.81" y="72.39"/>
 <element name="D2" library="JLY Parts" package="DO214AB" value="SK1035-TP" x="7.6962" y="15.24" smashed="yes" rot="R180">
-<attribute name="NAME" x="1.5494" y="16.383" size="1.27" layer="21" rot="SR270"/>
+<attribute name="NAME" x="6.9342" y="10.668" size="1.27" layer="21" rot="SR0"/>
 </element>
 <element name="D4" library="JLY Parts" package="DO214AB" value="SK1035-TP" x="40.767" y="18.542" smashed="yes" rot="R90">
@@
 <element name="U$3" library="SchmalzHausPublic" package="ROHS_GARBAGE_5MM" value="ROHS_GARBAGE" x="31.242" y="37.846"/>
 <element name="U$4" library="SchmalzHausPublic" package="ROHS_GARBAGE_5MM" value="" x="5.588" y="30.734" rot="MR90"/>
-<element name="U$5" library="SparkFun-Aesthetics" package="OSHW-LOGO-M" value="" x="8.636" y="39.878" rot="MR90"/>
+<element name="LOGO3" library="SparkFun-Aesthetics" package="OSHW-LOGO-M" value="OSHW-LOGOM" x="8.382" y="38.1" rot="MR90"/>
 </elements>
 <signals>
